Commit message: big
big robot based on FR-09

File: description/gazebo_control.xacro (robot description, xacro)
@@ -4,8 +4,8 @@
         <plugin name="diff_drive" filename="libgazebo_ros_diff_drive.so">
             <!-- Wheel Information -->
-            <left_joint>left_wheel_joint</left_joint>
-            <right_joint>right_wheel_joint</right_joint>
-            <wheel_separation>0.297</wheel_separation>
-            <wheel_diameter>0.066</wheel_diameter>
+            <left_joint>rear_left_wheel_joint</left_joint>
+            <right_joint>rear_right_wheel_joint</right_joint>
+            <wheel_separation>0.645</wheel_separation>
+            <wheel_diameter>0.420</wheel_diameter>
             <!-- Limits -->
             <max_wheel_torque>200</max_wheel_torque>

File: description/ros2_control.xacro (robot description, xacro)
@@ -5,6 +5,6 @@
             <hardware>
                 <plugin>diffdrive_arduino/DiffDriveArduino</plugin>
-                <param name="left_wheel_name">left_wheel_joint</param>
-                <param name="right_wheel_name">right_wheel_joint</param>
+                <param name="left_wheel_name">rear_left_wheel_joint</param>
+                <param name="right_wheel_name">rear_right_wheel_joint</param>
                 <param name="loop_rate">30</param>
                 <param name="device">/dev/ttyUSB0</param>
@@ -36,5 +36,5 @@
                 <plugin>gazebo_ros2_control/GazeboSystem</plugin>
             </hardware>
-            <joint name="left_wheel_joint">
+            <joint name="rear_left_wheel_joint">
                 <command_interface name="velocity">
                     <param name="min">-10</param>
@@ -44,5 +44,5 @@
                 <state_interface name="position"/>
             </joint>
-            <joint name="right_wheel_joint">
+            <joint name="rear_right_wheel_joint">
                 <command_interface name="velocity">
                     <param name="min">-10</param>
