Commit message: update steerbot

File: description/steer_bot.urdf.xacro (robot description, xacro)
@@ -17,4 +17,5 @@
   <!-- Include xacro for inertials, materials and wheels -->
   <xacro:include filename="$(find steer_bot_description)/urdf/wheel.xacro"/>
+  <xacro:include filename="$(find steer_bot_description)/urdf/lidar.xacro"/>
   <xacro:property name="robot_namespace" value="/steer_bot"/>
   <!-- Gazebo plugins -->
@@ -31,11 +32,11 @@
   <xacro:property name="deg_to_rad" value="0.01745329251994329577"/>
   <!-- Robot base dimensions -->
-  <xacro:property name="base_length" value="0.5" />
-  <xacro:property name="base_width" value="0.3" />
-  <xacro:property name="base_height" value="0.1" />
-  <xacro:property name="base_mass" value="5" />
+  <xacro:property name="base_length" value="1.4" />
+  <xacro:property name="base_width" value="0.618" />
+  <xacro:property name="base_height" value="0.287" />
+  <xacro:property name="base_mass" value="2.0" />
   <!-- Wheel link dimensions -->
-  <xacro:property name="wheel_radius" value="0.1" />
-  <xacro:property name="wheel_thickness" value="0.08" />
+  <xacro:property name="wheel_radius" value="0.21" />
+  <xacro:property name="wheel_thickness" value="0.130" />
   <xacro:property name="wheel_mass" value="1" />
   <!-- Steering link dimensions -->
@@ -44,7 +45,8 @@
   <xacro:property name="steer_mass" value="1" />
   <!-- Axle positions -->
-  <xacro:property name="axle_offset" value="0.05" />
+  <xacro:property name="axle_offset" value="0.065" /> <!-- track width (width of body)-->
   <xacro:property name="steer_offset" value="0.02" />
-  <!-- Base link -->
+  <xacro:property name="x_axle_offset" value="0.2" /> <!-- track lenght (length of body)-->
+  <!-- Base link, the chasis -->
   <link name="base_link">
     <visual>
@@ -66,4 +68,12 @@
         x="${base_length}" y="${base_width}" z="${base_height}" />
   </link>
+  <!-- BASE_FOOTPRINT LINK -->
+  <joint name="base_footprint_joint" type="fixed">
+    <parent link="base_link"/>
+    <child link="base_footprint"/>
+    <origin xyz="0 0 0" rpy="0 0 0"/>
+  </joint>
+  <link name="base_footprint">
+  </link>
   <!-- Front steer and rear wheel joints required for ackermann_steering_controller -->
   <xacro:front_steer
@@ -84,5 +94,5 @@
     wheel_thickness="${wheel_thickness/2}"
     wheel_mass="${wheel_mass/32}">
-    <origin xyz="${-base_length/2+axle_offset} 0 0" rpy="${-90 * deg_to_rad} 0 0"/>
+    <origin xyz="${-base_length/2+x_axle_offset} ${-base_width/2+axle_offset} ${-base_height/2}" rpy="${-90 * deg_to_rad} 0 0"/>
   </xacro:rear_wheel>
   <!-- Steerable front wheels -->
@@ -101,4 +111,5 @@
     axle_offset="${axle_offset}"
     steer_height="${wheel_radius+steer_offset}">
+    <origin xyz="${-base_length/2+axle_offset+base_length/2-x_axle_offset} 0 ${-base_height/2-wheel_radius-steer_offset}" rpy="${-90 * deg_to_rad} 0 0"/>
   </xacro:front_wheel_lr>
   <xacro:front_wheel_lr
@@ -116,4 +127,5 @@
     axle_offset="${axle_offset}"
     steer_height="${wheel_radius+steer_offset}">
+    <origin xyz="${-base_length/2+axle_offset+base_length/2-x_axle_offset} 0 ${-base_height/2-wheel_radius-steer_offset}" rpy="${-90 * deg_to_rad} 0 0"/>
   </xacro:front_wheel_lr>
   <!-- Rear wheels -->
@@ -124,5 +136,5 @@
     wheel_thickness="${wheel_thickness}"
     wheel_mass="${wheel_mass}">
-    <origin xyz="${-base_length/2+axle_offset} ${-base_width/2-axle_offset} 0" rpy="${-90 * deg_to_rad} 0 0"/>
+    <origin xyz="${-base_length/2+x_axle_offset} ${-base_width/2-axle_offset} ${-base_height/2}" rpy="${-90 * deg_to_rad} 0 0"/>
   </xacro:rear_wheel_lr>
   <xacro:rear_wheel_lr
@@ -132,5 +144,5 @@
     wheel_thickness="${wheel_thickness}"
     wheel_mass="${wheel_mass}">
-    <origin xyz="${-base_length/2+axle_offset} ${+base_width/2+axle_offset} 0" rpy="${-90 * deg_to_rad} 0 0"/>
+    <origin xyz="${-base_length/2+x_axle_offset} ${+base_width/2+axle_offset} ${-base_height/2}" rpy="${-90 * deg_to_rad} 0 0"/>
   </xacro:rear_wheel_lr>
   <!-- Colour -->
