Commit message: change urdf
remain the original one in the ori file

File: description/robot_core.xacro (robot description, xacro)
@@ -1,17 +1,30 @@
 <?xml version="1.0"?>
 <robot xmlns:xacro="http://www.ros.org/wiki/xacro" >
-    <xacro:include filename="inertial_macros.xacro"/>
-    <xacro:property name="chassis_length" value="1.6"/>
-    <xacro:property name="chassis_width" value="0.82"/>
-    <xacro:property name="chassis_height" value="0.52"/>
-    <xacro:property name="chassis_mass" value="1.0"/>
+    <xacro:include filename="wheel.xacro"/>
+    <xacro:property name="chassis_length" value="1.4"/>
+    <xacro:property name="chassis_width" value="0.618"/>
+    <xacro:property name="chassis_height" value="0.287"/>
+    <xacro:property name="chassis_mass" value="2.0"/>
+    <!-- wheel link dimensions -->
     <xacro:property name="wheel_radius" value="0.210"/>
-    <xacro:property name="wheel_thickness" value="0.130"/>
-    <xacro:property name="wheel_mass" value="0.05"/>
-    <xacro:property name="wheel_offset_x" value="${chassis_length / 2}"/> <!-- Half of the new chassis length -->
-    <xacro:property name="wheel_offset_y" value="${chassis_width / 2 + wheel_thickness / 2 }"/> <!-- Half of the new chassis width -->
-    <xacro:property name="front_wheel_offset_x" value="${chassis_length / 4}"/> <!-- Half of the front chassis length -->
-    <xacro:property name="rear_wheel_offset_x" value="${-chassis_length / 4}"/> <!-- Half of the rear chassis length -->
-    <xacro:property name="wheel_offset_z" value="0.01"/>
+    <xacro:property name="wheel_thickness" value="0.121"/>
+    <xacro:property name="wheel_mass" value="0.5"/>
+    <!-- Steering link dimensions -->
+    <xacro:property name="steer_radius" value="0.05" />
+    <xacro:property name="steer_thickness" value="0.02" />
+    <xacro:property name="steer_mass" value="0.5" />
+    <!-- Axle positions -->
+    <xacro:property name="axle_offset" value="0.065" /> <!-- track width (width of body)-->
+    <xacro:property name="steer_offset" value="0.02" />
+    <xacro:property name="x_axle_offset" value="0.2" /> <!-- track lenght (length of body)-->
+    <!-- Half of the new chassis length
+    <xacro:property name="wheel_offset_x" value="${chassis_length / 2}"/>
+    Half of the new chassis width
+    <xacro:property name="wheel_offset_y" value="${chassis_width / 2 + wheel_thickness / 2 }"/>
+    Half of the front chassis length
+    <xacro:property name="front_wheel_offset_x" value="${chassis_length / 4}"/>
+    Half of the rear chassis length
+    <xacro:property name="rear_wheel_offset_x" value="${-chassis_length / 4}"/>
+    <xacro:property name="wheel_offset_z" value="0.01"/> -->
     <material name="white">
         <color rgba="1 1 1 1" />
@@ -31,4 +44,21 @@
     <!-- BASE LINK -->
     <link name="base_link">
+        <visual>
+            <origin xyz="0 0 0" rpy="0 0 0"/>
+            <geometry>
+                <box size="${base_length} ${base_width} ${base_height}"/>
+            </geometry>
+            <material name="green" />
+          </visual>
+          <collision>
+            <origin xyz="0 0 0" rpy="0 0 0"/>
+            <geometry>
+                <box size="${base_length} ${base_width} ${base_height}"/>
+            </geometry>
+          </collision>
+          <xacro:solid_cuboid_inertial
+                rpy="0 0 0" xyz="0 0 0"
+                mass="${base_mass}"
+                x="${base_length}" y="${base_width}" z="${base_height}" />
     </link>
     <!-- BASE_FOOTPRINT LINK -->
@@ -40,134 +70,77 @@
     <link name="base_footprint">
     </link>
-    <!-- CHASSIS LINK -->
-    <joint name="chassis_joint" type="fixed">
-        <parent link="base_link"/>
-        <child link="chassis"/>
-        <origin xyz="${-wheel_offset_x} 0 ${-wheel_offset_z}"/>
-    </joint>
-    <link name="chassis">
-        <visual>
-            <origin xyz="${chassis_length/2} 0 ${chassis_height/2}"/>
-            <geometry>
-                <box size="${chassis_length} ${chassis_width} ${chassis_height}"/>
-            </geometry>
-            <material name="orange"/>
-        </visual>
-        <collision>
-            <origin xyz="${chassis_length/2} 0 ${chassis_height/2}"/>
-            <geometry>
-                <box size="${chassis_length} ${chassis_width} ${chassis_height}"/>
-            </geometry>
-        </collision>
-        <xacro:inertial_box mass="0.5" x="${chassis_length}" y="${chassis_width}" z="${chassis_height}">
-            <origin xyz="${chassis_length/2} 0 ${chassis_height/2}" rpy="0 0 0"/>
-        </xacro:inertial_box>
-    </link>
-    <gazebo reference="chassis">
-        <material>Gazebo/Orange</material>
-    </gazebo>
-    <!-- LEFT WHEEL LINK -->
-    <joint name="front_left_wheel_joint" type="continuous">
-        <parent link="base_link"/>
-        <child link="front_left_wheel"/>
-        <origin xyz="${front_wheel_offset_x} ${wheel_offset_y} 0" rpy="-${pi/2} 0 0" />
-        <axis xyz="0 0 1"/>
-    </joint>
-    <link name="front_left_wheel">
-        <visual>
-            <geometry>
-                <cylinder radius="${wheel_radius}" length="${wheel_thickness}"/>
-            </geometry>
-            <material name="blue"/>
-        </visual>
-        <collision>
-            <geometry>
-                <sphere radius="${wheel_radius}"/>
-            </geometry>
-        </collision>
-        <xacro:inertial_cylinder mass="${wheel_mass}" length="${wheel_thickness}" radius="${wheel_radius}">
-            <origin xyz="0 0 0" rpy="0 0 0"/>
-        </xacro:inertial_cylinder>
-    </link>
-    <gazebo reference="front_left_wheel">
-        <material>Gazebo/Blue</material>
-    </gazebo>
-    <!-- RIGHT WHEEL LINK -->
-    <joint name="front_right_wheel_joint" type="continuous">
-        <parent link="base_link"/>
-        <child link="front_right_wheel"/>
-        <origin xyz="${front_wheel_offset_x} ${-wheel_offset_y} 0" rpy="${pi/2} 0 0" />
-        <axis xyz="0 0 -1"/>
-    </joint>
-    <link name="front_right_wheel">
-        <visual>
-            <geometry>
-                <cylinder radius="${wheel_radius}" length="${wheel_thickness}"/>
-            </geometry>
-            <material name="blue"/>
-        </visual>
-        <collision>
-            <geometry>
-                <sphere radius="${wheel_radius}"/>
-            </geometry>
-        </collision>
-        <xacro:inertial_cylinder mass="${wheel_mass}" length="${wheel_thickness}" radius="${wheel_radius}">
-            <origin xyz="0 0 0" rpy="0 0 0"/>
-        </xacro:inertial_cylinder>
-    </link>
-    <gazebo reference="front_right_wheel">
-        <material>Gazebo/Blue</material>
-    </gazebo>
-    <!-- REAR LEFT WHEEL LINK -->
-    <joint name="rear_left_wheel_joint" type="continuous">
-        <parent link="base_link"/>
-        <child link="rear_left_wheel"/>
-        <origin xyz="${rear_wheel_offset_x} ${wheel_offset_y} 0" rpy="-${pi/2} 0 0" />
-        <axis xyz="0 0 1"/>
-    </joint>
-    <link name="rear_left_wheel">
-        <visual>
-            <geometry>
-                <cylinder radius="${wheel_radius}" length="${wheel_thickness}"/>
-            </geometry>
-            <material name="blue"/>
-        </visual>
-        <collision>
-            <geometry>
-                <sphere radius="${wheel_radius}"/>
-            </geometry>
-        </collision>
-        <xacro:inertial_cylinder mass="${wheel_mass}" length="${wheel_thickness}" radius="${wheel_radius}">
-            <origin xyz="0 0 0" rpy="0 0 0"/>
-        </xacro:inertial_cylinder>
-    </link>
-    <gazebo reference="rear_left_wheel">
-        <material>Gazebo/Blue</material>
-    </gazebo>
-    <!-- REAR RIGHT WHEEL LINK -->
-    <joint name="rear_right_wheel_joint" type="continuous">
-        <parent link="base_link"/>
-        <child link="rear_right_wheel"/>
-        <origin xyz="${rear_wheel_offset_x} ${-wheel_offset_y} 0" rpy="-${pi/2} 0 0" />
-        <axis xyz="0 0 1"/>
-    </joint>
-    <link name="rear_right_wheel">
-        <visual>
-            <geometry>
-                <cylinder radius="${wheel_radius}" length="${wheel_thickness}"/>
-            </geometry>
-            <material name="blue"/>
-        </visual>
-        <collision>
-            <geometry>
-                <sphere radius="${wheel_radius}"/>
-            </geometry>
-        </collision>
-        <xacro:inertial_cylinder mass="${wheel_mass}" length="${wheel_thickness}" radius="${wheel_radius}">
-            <origin xyz="0 0 0" rpy="0 0 0"/>
-        </xacro:inertial_cylinder>
-    </link>
-    <gazebo reference="rear_right_wheel">
-        <material>Gazebo/Blue</material>
+    <!-- Front steer and rear wheel joints required for ackermann_steering_controller -->
+    <xacro:front_steer
+        name="front"
+        parent="base"
+        steer_radius="${steer_radius}"
+        steer_thickness="${steer_thickness}"
+        steer_mass="${steer_mass}"
+        base_length="${base_length}"
+        base_width="${base_width}"
+        axle_offset="${axle_offset}"
+        steer_height="${wheel_radius+steer_offset}">
+    </xacro:front_steer>
+    <xacro:rear_wheel
+        name="rear"
+        parent="base"
+        wheel_radius="${wheel_radius/4}"
+        wheel_thickness="${wheel_thickness/2}"
+        wheel_mass="${wheel_mass/32}">
+        <origin xyz="${-base_length/2+x_axle_offset} ${-base_width/2+axle_offset} ${-base_height/2}" rpy="${-90 * deg_to_rad} 0 0"/>
+    </xacro:rear_wheel>
+    <!-- Steerable front wheels -->
+    <xacro:front_wheel_lr
+        name="front_right"
+        parent="base"
+        reflect="-1"
+        wheel_radius="${wheel_radius}"
+        wheel_thickness="${wheel_thickness}"
+        wheel_mass="${wheel_mass}"
+        steer_radius="${steer_radius}"
+        steer_thickness="${steer_thickness}"
+        steer_mass="${steer_mass}"
+        base_length="${base_length}"
+        base_width="${base_width}"
+        axle_offset="${axle_offset}"
+        steer_height="${wheel_radius+steer_offset}">
+        <origin xyz="${-base_length/2+axle_offset+base_length/2-x_axle_offset} 0 ${-base_height/2-wheel_radius-steer_offset}" rpy="${-90 * deg_to_rad} 0 0"/>
+    </xacro:front_wheel_lr>
+    <xacro:front_wheel_lr
+        name="front_left"
+        parent="base"
+        reflect="1"
+        wheel_radius="${wheel_radius}"
+        wheel_thickness="${wheel_thickness}"
+        wheel_mass="${wheel_mass}"
+        steer_radius="${steer_radius}"
+        steer_thickness="${steer_thickness}"
+        steer_mass="${steer_mass}"
+        base_length="${base_length}"
+        base_width="${base_width}"
+        axle_offset="${axle_offset}"
+        steer_height="${wheel_radius+steer_offset}">
+    <origin xyz="${-base_length/2+axle_offset+base_length/2-x_axle_offset} 0 ${-base_height/2-wheel_radius-steer_offset}" rpy="${-90 * deg_to_rad} 0 0"/>
+    </xacro:front_wheel_lr>
+    <!-- Rear wheels -->
+    <xacro:rear_wheel_lr
+        name="rear_right"
+        parent="base"
+        wheel_radius="${wheel_radius}"
+        wheel_thickness="${wheel_thickness}"
+        wheel_mass="${wheel_mass}">
+        <origin xyz="${-base_length/2+x_axle_offset} ${-base_width/2-axle_offset} ${-base_height/2}" rpy="${-90 * deg_to_rad} 0 0"/>
+    </xacro:rear_wheel_lr>
+    <xacro:rear_wheel_lr
+        name="rear_left"
+        parent="base"
+        wheel_radius="${wheel_radius}"
+        wheel_thickness="${wheel_thickness}"
+        wheel_mass="${wheel_mass}">
+        <origin xyz="${-base_length/2+x_axle_offset} ${+base_width/2+axle_offset} ${-base_height/2}" rpy="${-90 * deg_to_rad} 0 0"/>
+    </xacro:rear_wheel_lr>
+    <!-- Colour -->
+    <gazebo reference="base_link">
+        <material>Gazebo/Green</material>
     </gazebo>
 </robot>

Commit message: delete unused

File: description/robot_core.xacro (robot description, xacro)
@@ -18,28 +18,4 @@
     <xacro:property name="steer_offset" value="0.02" />
     <xacro:property name="x_axle_offset" value="0.2" /> <!-- track lenght (length of body)-->
-    <!-- Half of the new chassis length
-    <xacro:property name="wheel_offset_x" value="${chassis_length / 2}"/>
-    Half of the new chassis width
-    <xacro:property name="wheel_offset_y" value="${chassis_width / 2 + wheel_thickness / 2 }"/>
-    Half of the front chassis length
-    <xacro:property name="front_wheel_offset_x" value="${chassis_length / 4}"/>
-    Half of the rear chassis length
-    <xacro:property name="rear_wheel_offset_x" value="${-chassis_length / 4}"/>
-    <xacro:property name="wheel_offset_z" value="0.01"/> -->
-    <material name="white">
-        <color rgba="1 1 1 1" />
-    </material>
-    <material name="orange">
-        <color rgba="1 0.3 0.1 1"/>
-    </material>
-    <material name="blue">
-        <color rgba="0.2 0.2 1 1"/>
-    </material>
-    <material name="black">
-        <color rgba="0 0 0 1"/>
-    </material>
-    <material name="red">
-        <color rgba="1 0 0 1"/>
-    </material>
     <!-- BASE LINK -->
     <link name="base_link">
