Commit message: lidar and camera reposition

File: description/camera.xacro (robot description, xacro)
@@ -4,5 +4,5 @@
         <parent link="chassis"/>
         <child link="camera_link"/>
-        <origin xyz="0.276 0 0.181" rpy="0 0.18 0"/>
+        <origin xyz="1.541 0 0.563" rpy="0 0.18 0"/>
     </joint>
     <link name="camera_link">

File: description/lidar.xacro (robot description, xacro)
@@ -4,5 +4,5 @@
         <parent link="chassis"/>
         <child link="laser_frame"/>
-        <origin xyz="0.122 0 0.212" rpy="0 0 0"/>
+        <origin xyz="0.122 0 0.594" rpy="0 0 0"/>
     </joint>
     <link name="laser_frame">

Commit message: revert ori

File: description/camera.xacro (robot description, xacro)
@@ -4,5 +4,5 @@
         <parent link="chassis"/>
         <child link="camera_link"/>
-        <origin xyz="1.541 0 0.563" rpy="0 0.18 0"/>
+        <origin xyz="0.276 0 0.181" rpy="0 0.18 0"/>
     </joint>
     <link name="camera_link">

File: description/lidar.xacro (robot description, xacro)
@@ -4,5 +4,5 @@
         <parent link="chassis"/>
         <child link="laser_frame"/>
-        <origin xyz="0.122 0 0.594" rpy="0 0 0"/>
+        <origin xyz="0.122 0 0.212" rpy="0 0 0"/>
     </joint>
     <link name="laser_frame">

Commit message: change chassis to base_link

File: description/camera.xacro (robot description, xacro)
@@ -2,5 +2,5 @@
 <robot xmlns:xacro="http://www.ros.org/wiki/xacro" >
     <joint name="camera_joint" type="fixed">
-        <parent link="chassis"/>
+        <parent link="base"/>
         <child link="camera_link"/>
         <origin xyz="1.541 0 0.563" rpy="0 0.18 0"/>

File: description/depth_camera.xacro (robot description, xacro)
@@ -2,5 +2,5 @@
 <robot xmlns:xacro="http://www.ros.org/wiki/xacro" >
     <joint name="camera_joint" type="fixed">
-        <parent link="chassis"/>
+        <parent link="base"/>
         <child link="camera_link"/>
         <origin xyz="0.305 0 0.08" rpy="0 0 0"/>

File: description/face.xacro (robot description, xacro)
@@ -2,7 +2,7 @@
 <robot xmlns:xacro="http://www.ros.org/wiki/xacro" >
     <joint name="face_joint" type="fixed">
-        <parent link="chassis"/>
+        <parent link="base"/>
         <child link="face_link"/>
-        <origin xyz="${chassis_length} 0 ${chassis_height/2}" rpy="0 0 0"/>
+        <origin xyz="${base} 0 ${base_height/2}" rpy="0 0 0"/>
     </joint>
     <link name="face_link">

File: description/lidar.xacro (robot description, xacro)
@@ -2,5 +2,5 @@
 <robot xmlns:xacro="http://www.ros.org/wiki/xacro" >
     <joint name="laser_joint" type="fixed">
-        <parent link="chassis"/>
+        <parent link="base"/>
         <child link="laser_frame"/>
         <origin xyz="0.122 0 0.594" rpy="0 0 0"/>

File: description/robot_core.xacro (robot description, xacro)
@@ -2,8 +2,8 @@
 <robot xmlns:xacro="http://www.ros.org/wiki/xacro" >
     <xacro:include filename="wheel.xacro"/>
-    <xacro:property name="chassis_length" value="1.4"/>
-    <xacro:property name="chassis_width" value="0.618"/>
-    <xacro:property name="chassis_height" value="0.287"/>
-    <xacro:property name="chassis_mass" value="2.0"/>
+    <xacro:property name="base_length" value="1.4"/>
+    <xacro:property name="base_width" value="0.618"/>
+    <xacro:property name="base_height" value="0.287"/>
+    <xacro:property name="base_mass" value="2.0"/>
     <!-- wheel link dimensions -->
     <xacro:property name="wheel_radius" value="0.210"/>
